File: nRF52Buddy.kicad_sch (KiCad schematic)
At the start: 4 parts

Commit message: Updates for revision 3
Other:
- sheet Connectors ports: added P0.13/STATUS_LED4, P0.26/V_USB_CONNECTED, P1.09, P1.10/STATUS_LED1, P1.11/STATUS_LED2, P1.12/STATUS_LED3; removed P0.13, P0.26, P1.09/~{CHARGE}, P1.10, P1.11, P1.12
- sheet MCU (nRF52840) ports: added P0.13/STATUS_LED4, P1.09; removed P0.13/BT_STATUS_LED, P1.09/~{CHARGE}
Changed lines of the file:
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@@
   (title_block
     (title "nRF Buddy Board Schematic")
-    (rev "2")
+    (rev "3")
     (company "Kane Stoboi")
   )
@@
   )
   (wire (pts (xy 191.77 88.9) (xy 217.17 88.9))
-    (stroke (width 0) (type default))
-  )
-  (wire (pts (xy 46.99 83.82) (xy 62.23 83.82))
     (stroke (width 0) (type default))
   )
@@
     (effects (font (size 1.27 1.27)) (justify right bottom))
   )
-  (label "P1.09{slash}~{CHARGE}" (at 196.85 123.19 0) (fields_autoplaced)
-    (effects (font (size 1.27 1.27)) (justify left bottom))
-  )
   (label "SCL" (at 60.96 53.34 180) (fields_autoplaced)
     (effects (font (size 1.27 1.27)) (justify right bottom))
   )
   (label "SCL" (at 200.66 33.02 180) (fields_autoplaced)
-    (effects (font (size 1.27 1.27)) (justify right bottom))
-  )
-  (label "P1.09{slash}~{CHARGE}" (at 62.23 83.82 180) (fields_autoplaced)
     (effects (font (size 1.27 1.27)) (justify right bottom))
   )
@@
       (effects (font (size 1.27 1.27)) (justify left top))
     )
-    (pin "P1.10" bidirectional (at 217.17 125.73 180)
-      (effects (font (size 1.27 1.27)) (justify left))
-    )
-    (pin "P1.12" bidirectional (at 217.17 130.81 180)
-      (effects (font (size 1.27 1.27)) (justify left))
-    )
-    (pin "P1.11" bidirectional (at 217.17 128.27 180)
-      (effects (font (size 1.27 1.27)) (justify left))
-    )
-    (pin "P0.26" input (at 217.17 83.82 180)
-      (effects (font (size 1.27 1.27)) (justify left))
-    )
-    (pin "P0.13" bidirectional (at 217.17 50.8 180)
+    (pin "P1.10{slash}STATUS_LED1" bidirectional (at 217.17 125.73 180)
+      (effects (font (size 1.27 1.27)) (justify left))
+    )
+    (pin "P1.12{slash}STATUS_LED3" bidirectional (at 217.17 130.81 180)
+      (effects (font (size 1.27 1.27)) (justify left))
+    )
+    (pin "P1.11{slash}STATUS_LED2" bidirectional (at 217.17 128.27 180)
+      (effects (font (size 1.27 1.27)) (justify left))
+    )
+    (pin "P0.26{slash}V_USB_CONNECTED" input (at 217.17 83.82 180)
+      (effects (font (size 1.27 1.27)) (justify left))
+    )
+    (pin "P0.13{slash}STATUS_LED4" bidirectional (at 217.17 50.8 180)
       (effects (font (size 1.27 1.27)) (justify left))
     )
@@
       (effects (font (size 1.27 1.27)) (justify left))
     )
-    (pin "P1.09{slash}~{CHARGE}" input (at 217.17 123.19 180)
+    (pin "P1.09" input (at 217.17 123.19 180)
       (effects (font (size 1.27 1.27)) (justify left))
     )
@@
       (effects (font (size 1.27 1.27)) (justify right))
     )
-    (pin "P1.09{slash}~{CHARGE}" input (at 191.77 123.19 0)
+    (pin "P1.09" input (at 191.77 123.19 0)
       (effects (font (size 1.27 1.27)) (justify right))
     )
@@
       (effects (font (size 1.27 1.27)) (justify left))
     )
-    (pin "P0.13{slash}BT_STATUS_LED" bidirectional (at 191.77 50.8 0)
-      (effects (font (size 1.27 1.27)) (justify right))
-    )
+    (pin "P0.13{slash}STATUS_LED4" bidirectional (at 191.77 50.8 0)
+      (effects (font (size 1.27 1.27)) (justify right))
+    )
