File: Sheets/2_power_input.kicad_sch (KiCad schematic)
At the start: 20 parts, among them J1 2060-452_998-404, J6 S2B-PH-SM4-TB(LF)(SN), Q1 SSM3J332R, Q4 SSM3J332R, U1 AP9211, U2 MAX17260SETD, U3 TP4054

Commit message: Updates for revision 2
Parts:
- removed D13: 12V Status LED, LED_SMD:LED_0805_2012Metric, symbol Device:LED
- removed Q4: SSM3J332R, Package_TO_SOT_SMD:SOT-23, symbol Device:Q_PMOS_GSD
- removed R22: 1k5, Resistor_SMD:R_0402_1005Metric, symbol Device:R
- removed R30: 10k, Resistor_SMD:R_0402_1005Metric, symbol Device:R
- D1: MANUFACTURER (none) -> TECH PUBLIC; MAXIMUM_PACKAGE_HEIGHT TECH PUBLIC -> (none)
- J1: footprint SnapEDA Library:WAGO_2060-452_998-404 -> Footprints:WAGO_2060-452_998-404
- J6: value S2B-PH-SM4-TB(LF)(SN) -> HDGC1251WR-S-2P; footprint Footprints:JST_S2B-PH-SM4-TB(LF)(SN) -> Footprints:HDGC1251WR-S-2P; MANUFACTURER JST -> HDGC; Manufacturer Part Number HDGC2001WR-S-2P -> HDGC1251WR-S-2P
- R32: value 10k -> 1k5; Manufacturer Part Number 0402WGF1002TCE -> 0402WGF1501TCE
Connections:
- net BATT_IN is gone; now on net BATT_CONN+: C3.1, R2.2, U2.6 (BATT), U2.7 (CSN)
- net VCC is gone; now on net BATT_CONN+: C4.1, U1.3 (VDD)
- net +12V_CONN: now also D1.1 (A1); no longer D1.2 (A2)
- net +5V: no longer R32.2
- net BATT+: now also U3.3 (BATT)
- net BATT_CONN+: no longer U3.3 (BATT)
- net GND: now also D1.2 (A2); no longer D1.1 (A1)
- net ~{CHARGE} renamed P1.09/~{CHARGE}
- new net +3V3: R32.2
Other:
- note added: "For I_{CHARGE} <= 0.15A R_{PROG} = 1000/I_{BAT} R_{PROG} = = 1000/0.1 R_{PROG} = 10k"
- note removed: "For I_{BAT} <= 0.15A R_{PROG} = 1000/I_{BAT} R_{PROG} = = 1000/0.1 R_{PROG} = 10k"
- moved on the sheet: C4, D1, J1, Q1

Commit message: Updating bom with datasheets, manufactures, and part numbers
Parts:
- C26, C3, C4, C5: MANUFACTURER (none) -> Samsung Electro-Mechanics
- D1: MANUFACTURER TECH PUBLIC -> Nexperia; Manufacturer Part Number pesd5v0l1ba -> PESD5V0L1BA,115
- D16: MANUFACTURER (none) -> Orient
- J1: MAXIMUM_PACKAGE_HEIGHT 4.5 mm -> (none); Manufacturer Part Number 2060-452_998-404 -> 2060-452/998-404; PARTREV N/A -> (none); SNAPEDA_PN 2060-452/998-404 -> (none); STANDARD Manufacturer Recommendations -> (none)
- J6: STANDARD Manufacturer Recommendation -> (none)
- Q1: Manufacturer Part Number SSM3J332R -> SSM3J332R,LF
- R1: MANUFACTURER (none) -> Royalohm
- U1: MANUFACTURER (none) -> Diodes Incorporated; Manufacturer Part Number AP9211 -> AP9211SA-AK-HAC-7
- U2: MANUFACTURER (none) -> Maxim Integrated; Manufacturer Part Number MAX17260SETD -> MAX17260SETD+
- U3: MANUFACTURER (none) -> TECH PUBLIC

Commit message: updating bom
Parts:
- D1: value D_TVS -> D_TVS_15V; Manufacturer Part Number PESD5V0L1BA,115 -> PESD15VL1BA,115
Changed lines of the file:
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@@
       (effects (font (size 1.27 1.27)) (justify left))
     )
-    (property "Value" "D_TVS" (at 76.2 166.3699 90)
+    (property "Value" "D_TVS_15V" (at 76.2 166.3699 90)
       (effects (font (size 1.27 1.27)) (justify left))
     )
@@
       (effects (font (size 1.27 1.27)) hide)
     )
-    (property "Manufacturer Part Number" "PESD5V0L1BA,115" (at 73.66 165.1 0)
+    (property "Manufacturer Part Number" "PESD15VL1BA,115" (at 73.66 165.1 0)
       (effects (font (size 1.27 1.27)) hide)
     )
@@
       (effects (font (size 1.27 1.27)) (justify left))
     )
-    (property "Value" "HDGC1251WR-S-2P" (at 27.94 73.66 0)
+    (property "Value" "HDGC1251WR-S-2P" (at 49.53 73.66 0)
       (effects (font (size 1.27 1.27)) (justify left))
     )

Commit message: Moving some tracks and increasing via diameter to allow for latest JLCPCB capabilities
Parts:
- U1: footprint AP9211SA-AK-HAC-7:DFN200X300X60-7N -> Footprints:DFN200X300X60-7N
Changed lines of the file:
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@@
       (effects (font (size 1.27 1.27)))
     )
-    (property "Footprint" "AP9211SA-AK-HAC-7:DFN200X300X60-7N" (at 109.22 115.57 0)
+    (property "Footprint" "Footprints:DFN200X300X60-7N" (at 109.22 115.57 0)
       (effects (font (size 1.27 1.27)) hide)
     )

Commit message: Updates for revision 3
Connections:
- net +3V3 is gone; now on net +5V: R32.2
- net BATT_CONN+: now also U2.1 (TH)
- net GND: now also U2.9 (CSPL)
- net P1.09/~{CHARGE}: no longer names the net of D16.1 (K), U3.1 (~{CHARGE})
- no-connect marks 4 -> 2
Changed lines of the file:
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@@
   (title_block
     (title "Power Input")
-    (rev "2")
+    (rev "3")
     (company "Kane Stoboi")
   )
@@
   (junction (at 139.7 118.11) (diameter 0) (color 0 0 0 0)
   )
+  (junction (at 191.77 129.54) (diameter 0) (color 0 0 0 0)
+  )
+  (junction (at 208.28 138.43) (diameter 0) (color 0 0 0 0)
+  )
   (junction (at 109.22 45.72) (diameter 0) (color 0 0 0 0)
   )
@@
   (junction (at 168.91 77.47) (diameter 0) (color 0 0 0 0)
   )
-  (junction (at 153.67 43.18) (diameter 0) (color 0 0 0 0)
-  )
   (junction (at 107.95 38.1) (diameter 0) (color 0 0 0 0)
   )
@@
   (junction (at 97.79 121.92) (diameter 0) (color 0 0 0 0)
   )
-  (no_connect (at 198.12 132.08))
   (no_connect (at 198.12 116.84))
   (no_connect (at 48.26 85.09))
-  (no_connect (at 198.12 124.46))
   (polyline (pts (xy 83.82 92.71) (xy 149.86 92.71))
     (stroke (width 0) (type default))
@@
     (stroke (width 0) (type default))
   )
+  (wire (pts (xy 208.28 138.43) (xy 208.28 139.7))
+    (stroke (width 0) (type default))
+  )
   (wire (pts (xy 190.5 71.12) (xy 190.5 77.47))
     (stroke (width 0) (type default))
@@
     (stroke (width 0) (type default))
   )
-  (wire (pts (xy 153.67 43.18) (xy 160.02 43.18))
+  (wire (pts (xy 208.28 138.43) (xy 208.28 137.16))
+    (stroke (width 0) (type default))
+  )
+  (wire (pts (xy 191.77 124.46) (xy 191.77 129.54))
     (stroke (width 0) (type default))
   )
@@
     (stroke (width 0) (type default))
   )
+  (wire (pts (xy 191.77 129.54) (xy 168.91 129.54))
+    (stroke (width 0) (type default))
+  )
   (wire (pts (xy 62.23 20.32) (xy 62.23 71.12))
     (stroke (width 0) (type default))
@@
     (stroke (width 0) (type default))
   )
-  (wire (pts (xy 153.67 26.67) (xy 153.67 43.18))
-    (stroke (width 0) (type default))
-  )
   (wire (pts (xy 208.28 101.6) (xy 208.28 111.76))
     (stroke (width 0) (type default))
@@
     (stroke (width 0) (type default))
   )
-  (wire (pts (xy 134.62 43.18) (xy 153.67 43.18))
+  (wire (pts (xy 134.62 43.18) (xy 160.02 43.18))
     (stroke (width 0) (type default))
   )
@@
     (stroke (width 0) (type default))
   )
+  (wire (pts (xy 198.12 132.08) (xy 198.12 138.43))
+    (stroke (width 0) (type default))
+  )
   (wire (pts (xy 134.62 45.72) (xy 139.7 45.72))
     (stroke (width 0) (type default))
@@
     (stroke (width 0) (type default))
   )
-  (wire (pts (xy 198.12 129.54) (xy 168.91 129.54))
-    (stroke (width 0) (type default))
-  )
-  (wire (pts (xy 208.28 137.16) (xy 208.28 138.43))
+  (wire (pts (xy 198.12 129.54) (xy 191.77 129.54))
     (stroke (width 0) (type default))
   )
@@
     (stroke (width 0) (type default))
   )
+  (wire (pts (xy 198.12 138.43) (xy 208.28 138.43))
+    (stroke (width 0) (type default))
+  )
   (wire (pts (xy 168.91 129.54) (xy 168.91 77.47))
     (stroke (width 0) (type default))
@@
     (stroke (width 0) (type default))
   )
-  (wire (pts (xy 160.02 26.67) (xy 153.67 26.67))
-    (stroke (width 0) (type default))
-  )
   (wire (pts (xy 97.79 121.92) (xy 97.79 127))
     (stroke (width 0) (type default))
   )
   (wire (pts (xy 185.42 77.47) (xy 190.5 77.47))
+    (stroke (width 0) (type default))
+  )
+  (wire (pts (xy 198.12 124.46) (xy 191.77 124.46))
     (stroke (width 0) (type default))
   )
@@
   (label "PROG" (at 134.62 45.72 0) (fields_autoplaced)
     (effects (font (size 1.27 1.27)) (justify left bottom))
-  )
-  (hierarchical_label "P1.09{slash}~{CHARGE}" (shape input) (at 160.02 26.67 0) (fields_autoplaced)
-    (effects (font (size 1.27 1.27)) (justify left))
   )
   (hierarchical_label "FUEL GAUGE ALERT" (shape input) (at 223.52 121.92 0) (fields_autoplaced)
@@
     )
   )
-  (symbol (lib_id "power:GND") (at 208.28 138.43 0) (unit 1)
-    (in_bom yes) (on_board yes) (dnp no) (fields_autoplaced)
-    (property "Reference" "#PWR0159" (at 208.28 144.78 0)
-      (effects (font (size 1.27 1.27)) hide)
-    )
-    (property "Value" "GND" (at 208.28 142.9925 0)
-      (effects (font (size 1.27 1.27)))
-    )
-    (property "Footprint" "" (at 208.28 138.43 0)
-      (effects (font (size 1.27 1.27)) hide)
-    )
-    (property "Datasheet" "" (at 208.28 138.43 0)
+  (symbol (lib_id "power:GND") (at 208.28 139.7 0) (unit 1)
+    (in_bom yes) (on_board yes) (dnp no)
+    (property "Reference" "#PWR0159" (at 208.28 146.05 0)
+      (effects (font (size 1.27 1.27)) hide)
+    )
+    (property "Value" "GND" (at 208.28 143.51 0)
+      (effects (font (size 1.27 1.27)))
+    )
+    (property "Footprint" "" (at 208.28 139.7 0)
+      (effects (font (size 1.27 1.27)) hide)
+    )
+    (property "Datasheet" "" (at 208.28 139.7 0)
       (effects (font (size 1.27 1.27)) hide)
     )
@@
     )
   )
+  (symbol (lib_id "power:+5V") (at 185.42 34.29 0) (unit 1)
+    (in_bom yes) (on_board yes) (dnp no) (fields_autoplaced)
+    (property "Reference" "#PWR05" (at 185.42 38.1 0)
+      (effects (font (size 1.27 1.27)) hide)
+    )
+    (property "Value" "+5V" (at 185.42 30.6855 0)
+      (effects (font (size 1.27 1.27)))
+    )
+    (property "Footprint" "" (at 185.42 34.29 0)
+      (effects (font (size 1.27 1.27)) hide)
+    )
+    (property "Datasheet" "" (at 185.42 34.29 0)
+      (effects (font (size 1.27 1.27)) hide)
+    )
+    (pin "1")
+    (instances
+      (project "nRF52Buddy"
+        (path "/f8009b5e-2814-48af-8478-16f2aae29be6/68dd5206-f59c-4f8c-876f-1a7cd0389797"
+          (reference "#PWR05") (unit 1)
+        )
+      )
+    )
+  )
   (symbol (lib_id "Device:LED") (at 163.83 43.18 0) (unit 1)
     (in_bom yes) (on_board yes) (dnp no)
@@
         )
       )
-    )
-  )
-  (symbol (lib_id "power:+3V3") (at 185.42 34.29 0) (unit 1)
-    (in_bom yes) (on_board yes) (dnp no) (fields_autoplaced)
-    (property "Reference" "#PWR0132" (at 185.42 38.1 0)
-      (effects (font (size 1.27 1.27)) hide)
-    )
-    (property "Value" "+3V3" (at 185.42 30.6855 0)
-      (effects (font (size 1.27 1.27)))
-    )
-    (property "Footprint" "" (at 185.42 34.29 0)
-      (effects (font (size 1.27 1.27)) hide)
-    )
-    (property "Datasheet" "" (at 185.42 34.29 0)
-      (effects (font (size 1.27 1.27)) hide)
-    )
-    (pin "1")
-    (instances
-      (project "nRF52Buddy"
-        (path "/f8009b5e-2814-48af-8478-16f2aae29be6/845162ad-409f-414e-965e-548bd8fa43dd"
-          (reference "#PWR0132") (unit 1)
-        )
-        (path "/f8009b5e-2814-48af-8478-16f2aae29be6/68dd5206-f59c-4f8c-876f-1a7cd0389797"
-          (reference "#PWR01") (unit 1)
-        )
-      )
