File: Sheets/3_usb_input.kicad_sch (KiCad schematic)
At the start: 4 parts, among them J3 2305018-2, U7 USBLC6-2SC6

Commit message: Updates for revision 2
Parts:
- J3: footprint SnapEDA Library:TE_2305018-2 -> Footprints:TE_2305018-2

Commit message: Updating bom with datasheets, manufactures, and part numbers
Parts:
- J3: PARTREV 6.0 -> (none); STANDRAD Manufacturer Recommendation -> (none)
- U7: MANUFACTURER (none) -> STMicroelectronics
Changed lines of the file:
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@@
+      (effects (font (size 1.27 1.27)) hide)
+    )
+    (property "Alternate MPN" "" (at 189.23 87.63 0)
+      (effects (font (size 1.27 1.27)) hide)
+    )
+    (property "Alternate Manufacturer" "" (at 189.23 87.63 0)
+      (effects (font (size 1.27 1.27)) hide)
+    )
+    (property "MANUFACTURER" "STMicroelectronics" (at 189.23 87.63 0)
       (effects (font (size 1.27 1.27)) hide)
     )
@@
       (effects (font (size 1.27 1.27)) hide)
     )
-    (property "Datasheet" "~" (at 60.96 74.93 0)
+    (property "Datasheet" "https://au.mouser.com/datasheet/2/1365/1-3044649.pdf" (at 60.96 74.93 0)
       (effects (font (size 1.27 1.27)) hide)
     )
@@
     )
     (property "MANUFACTURER" "UNI-ROYAL(Uniroyal Elec)" (at 60.96 74.93 0)
+      (effects (font (size 1.27 1.27)) hide)
+    )
+    (property "Alternate MPN" "" (at 60.96 74.93 0)
+      (effects (font (size 1.27 1.27)) hide)
+    )
+    (property "Alternate Manufacturer" "" (at 60.96 74.93 0)
       (effects (font (size 1.27 1.27)) hide)
     )
@@
       (effects (font (size 1.27 1.27)) (justify left bottom) hide)
     )
-    (property "Datasheet" "" (at 100.33 82.55 0)
-      (effects (font (size 1.27 1.27)) (justify left bottom) hide)
-    )
-    (property "STANDRAD" "Manufacturer Recommendation" (at 100.33 82.55 0)
-      (effects (font (size 1.27 1.27)) (justify left bottom) hide)
-    )
-    (property "PARTREV" "6.0" (at 100.33 82.55 0)
+    (property "Datasheet" "https://au.mouser.com/datasheet/2/418/7/ENG_CD_2305018_A2-2032147.pdf" (at 100.33 82.55 0)
       (effects (font (size 1.27 1.27)) (justify left bottom) hide)
     )
@@
     )
     (property "Manufacturer Part Number" "2305018-2" (at 100.33 82.55 0)
+      (effects (font (size 1.27 1.27)) hide)
+    )
+    (property "Alternate MPN" "" (at 100.33 82.55 0)
+      (effects (font (size 1.27 1.27)) hide)
+    )
+    (property "Alternate Manufacturer" "" (at 100.33 82.55 0)
       (effects (font (size 1.27 1.27)) hide)
     )
@@
       (effects (font (size 1.27 1.27)) hide)
     )
-    (property "Datasheet" "~" (at 139.7 74.93 0)
+    (property "Datasheet" "https://au.mouser.com/datasheet/2/1365/1-3044649.pdf" (at 139.7 74.93 0)
       (effects (font (size 1.27 1.27)) hide)
     )
@@
       (effects (font (size 1.27 1.27)) hide)
     )
+    (property "Alternate MPN" "" (at 139.7 74.93 0)
+      (effects (font (size 1.27 1.27)) hide)
+    )
+    (property "Alternate Manufacturer" "" (at 139.7 74.93 0)
+      (effects (font (size 1.27 1.27)) hide)
+    )
